Commit message: Minor config update

File: crs_support/urdf/crs.urdf.xacro (robot description, xacro)
@@ -29,5 +29,5 @@
         <origin rpy="0 0 3.14159249728" xyz="0 0 0.180920744391" />
         <axis xyz="0 0 1" />
-        <limit effort="330.0" lower="-4" upper="3.28" velocity="3.14" />
+        <limit effort="330.0" lower="-4.3" upper="3.28" velocity="3.14" />
         <dynamics damping="0.0" friction="0.0" />
     </joint>
@@ -406,5 +406,5 @@
     <link name="${prefix}camera_link" />
     <joint name="${prefix}camera_link_joint" type="fixed">
-        <origin xyz="0.0 0.0 0.0" rpy="1.57 -1.57 0"/>
+        <origin xyz="0.0 0.0 -0.005" rpy="1.57 -1.57 0"/>
         <parent link="${prefix}camera_link_optical"/>
         <child link="${prefix}camera_link"/>
